Commit message: human: Rescale based on anthropometry

File: robots/human_description/robots/human.urdf (robot description, URDF)
Before this commit: robot human_36dof_ISB_model, 37 links, 36 joints
Links:
- link left_foot: mass 1.13208 -> 0.9; geometry visual mesh filename=package://example-robot-data/robots/human_description/meshe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 scale=0.0067 0.0067 0.0067
- link left_hand: mass 0.56604 -> 0.45; geometry visual mesh filename=package://example-robot-data/robots/human_description/meshe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 scale=0.0061 0.0061 0.0061
- link left_lowerarm: mass 1.60378 -> 1.28; geometry visual mesh filename=package://example-robot-data/robots/human_description/meshe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 scale=0.0055 0.0055 0.0055; visual mesh filename=package://example-robot-data/robots/human_description/meshe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 scale=0.0064 0.0064 0.0064
- link left_lowerleg: mass 4.52832 -> 3.6; geometry visual mesh filename=package://example-robot-data/robots/human_description/meshe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 scale=0.0056 0.0056 0.0056; visual mesh filename=package://example-robot-data/robots/human_description/meshe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 scale=0.0063 0.0066 0.007
- link left_upperarm: mass 2.26416 -> 1.8; geometry visual mesh filename=package://example-robot-data/robots/human_description/meshe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 scale=0.0039 0.0039 0.0039; visual mesh filename=package://example-robot-data/robots/human_description/meshe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 scale=0.0063 0.006 0.0069
- link left_upperleg: mass 11.6038 -> 9.22; geometry visual mesh filename=package://example-robot-data/robots/human_description/meshe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 scale=0.0062 0.0064 0.0069
- link middle_abdomen: mass 2.73586 -> 12.25; geometry visual mesh filename=package://example-robot-data/robots/human_description/meshe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 scale=0.007 0.007 0.007; visual mesh filename=package://example-robot-data/robots/human_description/meshe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 scale=0.0074 0.0074 0.0074
- link middle_head: mass 6.32078 -> 5.03; geometry visual mesh filename=package://example-robot-data/robots/human_description/meshe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 scale=0.005 0.005 0.005; visual mesh filename=package://example-robot-data/robots/human_description/meshe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 scale=0.0056 0.0056 0.0056
- link middle_head_virtual: geometry 
- link middle_pelvis: mass 13.3963 -> 10.65; geometry visual mesh filename=package://example-robot-data/robots/human_description/meshe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 scale=0.0063 0.0058 0.0058
- link middle_thorax: mass 28.6794 -> 11.97; geometry 
- link right_foot: mass 1.13208 -> 0.9; geometry visual mesh filename=package://example-robot-data/robots/human_description/meshe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 scale=0.0067 0.0067 0.0067
- link right_hand: mass 0.56604 -> 0.45; geometry visual mesh filename=package://example-robot-data/robots/human_description/meshe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 scale=0.0061 0.0061 0.0061
- link right_lowerarm: mass 1.60378 -> 1.28; geometry visual mesh filename=package://example-robot-data/robots/human_description/meshe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 scale=0.0055 0.0055 0.0055; visual mesh filename=package://example-robot-data/robots/human_description/meshe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 scale=0.0064 0.0064 0.0064
- link right_lowerleg: mass 4.52832 -> 3.6; geometry visual mesh filename=package://example-robot-data/robots/human_description/meshe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 scale=0.0056 0.0056 0.0056; visual mesh filename=package://example-robot-data/robots/human_description/meshe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 scale=0.0063 0.0066 0.007
- link right_upperarm: mass 2.26416 -> 1.8; geometry visual mesh filename=package://example-robot-data/robots/human_description/meshe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 scale=0.0039 0.0039 0.0039; visual mesh filename=package://example-robot-data/robots/human_description/meshe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 scale=0.0063 0.006 0.0069
- link right_upperleg: mass 11.6038 -> 9.22; geometry visual mesh filename=package://example-robot-data/robots/human_description/meshe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 scale=0.0062 0.0064 0.0069
Joints:
- joint left_ankle_X: limit lower=-0.523598333 upper=0.785398 effort=20 velocity=0 -> lower=-0.523598333 upper=0.785398 effort=20 velocity=2.0
- joint left_ankle_Z: limit lower=-1.570795 upper=0.7853975 effort=126 velocity=0 -> lower=-1.570795 upper=0.7853975 effort=126 velocity=12.7; origin xyz=0 -0.43 0 rpy=0 -0 0 -> xyz=0 -0.44 0 rpy=0 -0 0
- joint left_clavicle_joint_X: limit lower=-1.0472 upper=0.314159 effort=0 velocity=0 -> lower=-1.0472 upper=0.349066 effort=100 velocity=14.0; origin xyz=0 0.33 0 rpy=0 -0 0 -> xyz=0 0.176 0 rpy=0 -0 0
- joint left_elbow_Y: limit lower=-3.14159 upper=0.2 effort=15 velocity=0 -> lower=-3.14159 upper=0.349066 effort=15 velocity=6.0
- joint left_elbow_Z: limit lower=0 upper=2.617991667 effort=77 velocity=0 -> lower=0 upper=2.617991667 effort=77 velocity=19.9; origin xyz=0 -0.274 0 rpy=0 -0 0 -> xyz=0 -0.276 0 rpy=0 -0 0
- joint left_hip_X: limit lower=-1.047196667 upper=1.570795 effort=190 velocity=0 -> lower=-1.047196667 upper=1.570795 effort=120 velocity=12.0
- joint left_hip_Y: limit lower=-1.047196667 upper=1.570795 effort=60 velocity=0 -> lower=-1.047196667 upper=1.570795 effort=60 velocity=12.0
- joint left_hip_Z: limit lower=-1.047196667 upper=3.14159 effort=190 velocity=0 -> lower=-1.047196667 upper=3.14159 effort=185 velocity=12.0; origin xyz=0.053 -0.075 -0.080 rpy=0 -0 0 -> xyz=0.023 -0.1 -0.082 rpy=0 -0 0
- joint left_knee: limit lower=0 upper=3.14159 effort=168 velocity=0 -> lower=0 upper=3.14159 effort=130 velocity=18.6; origin xyz=0 -0.43 0 rpy=0 -0 0 -> xyz=0. -0.439 0. rpy=0 -0 0
- joint left_shoulder_X: limit lower=-1.0472 upper=3.14159 effort=71 velocity=0 -> lower=-1.0472 upper=3.14159 effort=71 velocity=6.0
- joint left_shoulder_Y: limit lower=-1.5708 upper=3.14159 effort=0 velocity=0 -> lower=-1.5708 upper=3.14159 effort=52 velocity=6.0
- joint left_shoulder_Z: limit lower=-3.14159 upper=3.14159 effort=92 velocity=0 -> lower=-3.14159 upper=3.14159 effort=92 velocity=17.6; origin xyz=0.008 -0.073 -0.204 rpy=0 -0 0 -> xyz=0.008 -0.075 -0.21 rpy=0 -0 0
- joint left_wrist_X: limit lower=-0.785398 upper=0.785398 effort=0 velocity=0 -> lower=-0.785398 upper=0.785398 effort=100 velocity=6.0
- joint left_wrist_Z: limit lower=-1.5708 upper=1.5708 effort=185 velocity=0 -> lower=-1.5708 upper=1.5708 effort=185 velocity=25.0; origin xyz=0 -0.28 0 rpy=0 -0 0 -> xyz=0 -0.287 0 rpy=0 -0 0
- joint middle_cervical_X: limit lower=-1.5708 upper=1.5708 effort=0 velocity=0 -> lower=-1.5708 upper=1.5708 effort=100 velocity=8.7
- joint middle_cervical_Y: limit lower=-1.5708 upper=1.5708 effort=0 velocity=0 -> lower=-1.5708 upper=1.5708 effort=100 velocity=8.7
- joint middle_cervical_Z: limit lower=-1.5708 upper=1.5708 effort=0 velocity=0 -> lower=-1.5708 upper=1.5708 effort=100 velocity=8.7; origin xyz=0 0.33 0 rpy=0 -0 0 -> xyz=0 0.25 0 rpy=0 -0 0
- joint middle_lumbar_X: limit lower=-0.785398 upper=0.785398 effort=159 velocity=0 -> lower=-0.785398 upper=0.785398 effort=160 velocity=5.2
- joint middle_lumbar_Z: limit lower=-3.14159 upper=0.785398 effort=243 velocity=0 -> lower=-3.14159 upper=0.785398 effort=190 velocity=5.2
- joint middle_thoracic_X: limit lower=-1.0472 upper=1.0472 effort=159 velocity=0 -> lower=-1.0472 upper=1.0472 effort=190 velocity=5.2
- joint middle_thoracic_Y: limit lower=-1.0472 upper=1.0472 effort=159 velocity=0 -> lower=-1.0472 upper=1.0472 effort=185 velocity=2.0
- joint middle_thoracic_Z: limit lower=-1.0472 upper=0.392699 effort=159 velocity=0 -> lower=-1.0472 upper=0.392699 effort=190 velocity=5.2; origin xyz=0 0.15 0 rpy=0 -0 0 -> xyz=0 0.223 0 rpy=0 -0 0
- joint right_ankle_X: limit lower=-0.523598333 upper=0.785398 effort=20 velocity=0 -> lower=-0.523598333 upper=0.785398 effort=20 velocity=6.0
- joint right_ankle_Z: limit lower=-1.570795 upper=0.7853975 effort=126 velocity=0 -> lower=-1.570795 upper=0.7853975 effort=126 velocity=12.7; origin xyz=0 -0.43 0 rpy=0 -0 0 -> xyz=0 -0.44 0 rpy=0 -0 0
- joint right_clavicle_joint_X: limit lower=-0.392699 upper=1.0472 effort=0 velocity=0 -> lower=-0.349066 upper=1.0472 effort=100 velocity=14.0; origin xyz=0 0.33 0 rpy=0 -0 0 -> xyz=0 0.176 0 rpy=0 -0 0
- joint right_elbow_Y: limit lower=-0.2 upper=3.14159 effort=15 velocity=0 -> lower=-0.349066 upper=3.14159 effort=15 velocity=6.0
- joint right_elbow_Z: limit lower=0 upper=2.617991667 effort=77 velocity=0 -> lower=0 upper=2.617991667 effort=77 velocity=19.9; origin xyz=0 -0.274 0 rpy=0 -0 0 -> xyz=0 -0.276 0 rpy=0 -0 0
- joint right_hip_X: limit lower=-1.570795 upper=1.047196667 effort=190 velocity=0 -> lower=-1.570795 upper=1.047196667 effort=120 velocity=6.0
- joint right_hip_Y: limit lower=-1.570795 upper=1.047196667 effort=190 velocity=0 -> lower=-1.570795 upper=1.047196667 effort=60 velocity=6.0
- joint right_hip_Z: limit lower=-1.047196667 upper=3.14159 effort=190 velocity=0 -> lower=-1.047196667 upper=3.14159 effort=185 velocity=12.0; origin xyz=0.053 -0.075 -0.080 rpy=0 -0 0 -> xyz=0.023 -0.1 0.082 rpy=0 -0 0
- joint right_knee: limit lower=0 upper=3.14159 effort=168 velocity=0 -> lower=0 upper=3.14159 effort=130 velocity=18.6; origin xyz=0 -0.43 0 rpy=0 -0 0 -> xyz=0 -0.439 0 rpy=0 -0 0
- joint right_shoulder_X: limit lower=-1.0472 upper=3.14159 effort=71 velocity=0 -> lower=-1.0472 upper=3.14159 effort=71 velocity=6.0
- joint right_shoulder_Y: limit lower=-1.5708 upper=3.14159 effort=0 velocity=0 -> lower=-1.5708 upper=3.14159 effort=52 velocity=6.0
- joint right_shoulder_Z: limit lower=-3.14159 upper=3.14159 effort=0 velocity=0 -> lower=-3.14159 upper=3.14159 effort=92 velocity=17.6; origin xyz=0.008 -0.073 0.204 rpy=0 -0 0 -> xyz=0.008 -0.075 0.21 rpy=0 -0 0
- joint right_wrist_X: limit lower=-0.785398 upper=0.785398 effort=0 velocity=0 -> lower=-0.785398 upper=0.785398 effort=100 velocity=6.0
- joint right_wrist_Z: limit lower=-1.5708 upper=1.5708 effort=185 velocity=0 -> lower=-1.5708 upper=1.5708 effort=100 velocity=25.0; origin xyz=0 -0.28 0 rpy=0 -0 0 -> xyz=0 -0.287 0 rpy=0 -0 0
